Commit message: parrot xacro update + launch update

File: World/WorldWithDrone/src/urdf_drone/parrot.gazebo.xacro (robot description, xacro)
@@ -1,171 +1,62 @@
 <?xml version="1.0"?>
 <robot name="parrot" xmlns:xacro="http://ros.org/wiki/xacro">
-  <xacro:arg name="laser_visual"  default="false" />
-  <xacro:arg name="camera_visual" default="false"/>
-  <xacro:arg name="imu_visual"    default="false"/>
-  <!-- <xacro:include filename="$(find 41068_ignition_bringup)/urdf/wheel.urdf.xacro"/> -->
+  <!-- IMU on imu_link -->
   <gazebo reference="imu_link">
-    <sensor type="imu" name="imu">
+    <sensor name="imu" type="imu">
       <always_on>true</always_on>
-      <visualize>$(arg imu_visual)</visualize>
       <update_rate>100</update_rate>
-      <topic>model/husky/imu</topic>
+      <!-- publish as drone imu -->
+      <topic>/drone/imu</topic>
       <gz_frame_id>imu_link</gz_frame_id>
-      <imu>
-        <angular_velocity>
-          <x>
-            <noise type="gaussian">
-              <mean>0.0</mean>
-              <stddev>2e-4</stddev>
-              <bias_mean>0.0000075</bias_mean>
-              <bias_stddev>0.0000008</bias_stddev>
-            </noise>
-          </x>
-          <y>
-            <noise type="gaussian">
-              <mean>0.0</mean>
-              <stddev>2e-4</stddev>
-              <bias_mean>0.0000075</bias_mean>
-              <bias_stddev>0.0000008</bias_stddev>
-            </noise>
-          </y>
-          <z>
-            <noise type="gaussian">
-              <mean>0.0</mean>
-              <stddev>2e-4</stddev>
-              <bias_mean>0.0000075</bias_mean>
-              <bias_stddev>0.0000008</bias_stddev>
-            </noise>
-          </z>
-        </angular_velocity>
-        <linear_acceleration>
-          <x>
-            <noise type="gaussian">
-              <mean>0.0</mean>
-              <stddev>1.7e-2</stddev>
-              <bias_mean>0.1</bias_mean>
-              <bias_stddev>0.001</bias_stddev>
-            </noise>
-          </x>
-          <y>
-            <noise type="gaussian">
-              <mean>0.0</mean>
-              <stddev>1.7e-2</stddev>
-              <bias_mean>0.1</bias_mean>
-              <bias_stddev>0.001</bias_stddev>
-            </noise>
-          </y>
-          <z>
-            <noise type="gaussian">
-              <mean>0.0</mean>
-              <stddev>1.7e-2</stddev>
-              <bias_mean>0.1</bias_mean>
-              <bias_stddev>0.001</bias_stddev>
-            </noise>
-          </z>
-        </linear_acceleration>
-      </imu>
-      <plugin
-        filename="ignition-gazebo-imu-system"
-        name="ignition::gazebo::systems::Imu">
-      </plugin>
+      <visualize>false</visualize>
     </sensor>
-    <material>Gazebo/Grey</material>
   </gazebo>
-  <!-- Move base directly without faffing around with diff drive controllers -->
-  <gazebo>
-    <plugin
-      filename="ignition-gazebo-velocity-control-system"
-      name="ignition::gazebo::systems::VelocityControl">
-      <topic>model/husky/cmd_vel</topic>
-    </plugin>
-  </gazebo>
-  <!-- Publish odometry separately -->
-  <gazebo>
-    <plugin
-      filename="ignition-gazebo-odometry-publisher-system"
-      name="ignition::gazebo::systems::OdometryPublisher">
-      <topic>model/husky/odometry</topic>
-      <odom_publish_frequency>20</odom_publish_frequency>
-      <odom_frame>odom</odom_frame>
-      <robot_base_frame>base_link</robot_base_frame>
-    </plugin>
-  </gazebo>
-  <gazebo>
-    <plugin
-      filename="ignition-gazebo-joint-state-publisher-system"
-      name="ignition::gazebo::systems::JointStatePublisher">
-      <topic>model/husky/joint_states</topic>
-    </plugin>
-  </gazebo>
-  <!-- Lidar and cameras use the general Sensors plugin -->
-  <gazebo>
-    <plugin
-        filename="libignition-gazebo-sensors-system.so"
-        name="ignition::gazebo::systems::Sensors">
-    </plugin>
-  </gazebo>
+  <!-- LIDAR on base_scan (you already have this link) -->
   <gazebo reference="base_scan">
-    <material>Gazebo/FlatBlack</material>
-    <sensor type="gpu_lidar" name="lidar">
-      <pose relative_to='base_scan'>0 0 0 0 0 0</pose>
-      <visualize>$(arg laser_visual)</visualize>
-      <topic>model/husky/scan</topic>
-      <update_rate>10</update_rate>
+    <sensor name="lidar" type="ray">
+      <always_on>true</always_on>
+      <update_rate>15</update_rate>
+      <!-- publish as drone scan -->
+      <topic>/drone/scan</topic>
       <gz_frame_id>base_scan</gz_frame_id>
       <ray>
         <scan>
           <horizontal>
-            <samples>360</samples>
+            <samples>720</samples>
             <resolution>1</resolution>
-            <min_angle>0.0</min_angle>
-            <max_angle>6.28319</max_angle>
+            <min_angle>-3.14159</min_angle>
+            <max_angle>3.14159</max_angle>
           </horizontal>
         </scan>
         <range>
-          <min>0.2</min>
-          <max>40</max>
-          <resolution>0.015</resolution>
+          <min>0.15</min>
+          <max>20.0</max>
+          <resolution>0.01</resolution>
         </range>
-        <noise>
-          <type>gaussian</type>
-          <mean>0.0</mean>
-          <stddev>0.01</stddev>
-        </noise>
       </ray>
-      <always_on>true</always_on>
+      <visualize>false</visualize>
     </sensor>
   </gazebo>
+  <!-- Down/forward camera on camera_link -->
   <gazebo reference="camera_link">
-    <sensor name="rgbd_camera" type="rgbd_camera">
+    <sensor name="drone_cam" type="rgbd_camera">
+      <always_on>true</always_on>
+      <update_rate>10</update_rate>
+      <topic>/drone/camera</topic>
+      <gz_frame_id>camera_link</gz_frame_id>
       <camera>
-        <horizontal_fov>2.0944</horizontal_fov>
+        <horizontal_fov>1.047</horizontal_fov>
         <image>
-          <width>720</width>
+          <width>640</width>
           <height>480</height>
+          <format>R8G8B8</format>
         </image>
         <clip>
-          <near>0.1</near>
-          <far>40</far>
+          <near>0.2</near>
+          <far>20</far>
         </clip>
-        <!-- depth_camera near/far clip seems to be ignored for some reason -->
-        <!--    We're using Ignition Gazebo Fortress, which uses sdf format 1.9: http://sdformat.org/tutorials?tut=roadmap -->
-        <!--    This takes the depth_camera parameter with near / far clip http://sdformat.org/spec?ver=1.4&elem=sensor  -->
-        <!-- We also use ign sensors v6 ( run ls | grep libignition-sensors in /usr/lib/x86_64-linux-gnu)-->
-        <!-- Looking at the source code, the sdf sets HasDepthCamera() and corresponding HasDepthNearClip() & HasDepthFarClip() which are used in RgbdCameraSensor.cc, so this should work? -->
-        <!--    SDF description of Camera: https://github.com/gazebosim/sdformat/blob/sdf9/src/Camera.cc#L598-->
-        <!--    Camera sensor source code: https://github.com/gazebosim/gz-sensors/blob/ign-sensors6/src/RgbdCameraSensor.cc#L311  -->
-        <depth_camera>
-          <clip>
-            <near>0.4</near>
-            <far>10</far>
-          </clip>
-        </depth_camera>
       </camera>
-      <always_on>1</always_on>
-      <update_rate>3</update_rate> <!--10-->
-      <visualize>$(arg camera_visual)</visualize>
-      <topic>/model/husky/camera</topic>
-      <gz_frame_id>camera_link</gz_frame_id>
+      <!-- if Ignition publishes points for this camera, we can bridge them too -->
+      <visualize>false</visualize>
     </sensor>
   </gazebo>
