Commit message: for the night

File: src/description/urdf/parrot.urdf.xacro (robot description, xacro)
@@ -1,15 +1,17 @@
 <?xml version="1.0" ?>
 <robot name="parrot" xmlns:xacro="http://ros.org/wiki/xacro">
-  <!-- give the whole robot a model_name (used by parrot.gazebo.xacro) -->
+  <!-- model name that Gazebo plugins will use for topics: /model/<model_name>/... -->
   <xacro:arg name="model_name" default="drone1"/>
-  <!-- include the shared props and the gazebo extras from THIS package -->
+  <!-- include local xacros from this package -->
   <xacro:include filename="$(find description)/urdf/common_properties.urdf.xacro"/>
   <xacro:include filename="$(find description)/urdf/parrot.gazebo.xacro"/>
+  <!-- camera offsets -->
   <xacro:property name="r200_cam_rgb_px" value="0.005"/>
   <xacro:property name="r200_cam_rgb_py" value="0.018"/>
   <xacro:property name="r200_cam_rgb_pz" value="0.013"/>
   <xacro:property name="r200_cam_depth_offset" value="0.01"/>
-  <!-- Main link -->
+  <!-- ================= base_link ================= -->
   <link name="base_link">
+    <!-- inertia from original file -->
     <inertial>
       <origin xyz="0 0 0" rpy="0 0 0"/>
@@ -19,5 +21,12 @@
                izz="3.328e-3" />
     </inertial>
-    <!-- all meshes now come from description/meshes/... -->
+    <!-- SIMPLE COLLISION so it doesn't fall through the world -->
+    <collision name="collision">
+      <origin xyz="0 0 0" rpy="0 0 0"/>
+      <geometry>
+        <box size="0.4 0.4 0.15"/>
+      </geometry>
+    </collision>
+    <!-- visuals (using your meshes copied into description/meshes) -->
     <visual name="hull">
       <geometry>
@@ -50,4 +59,5 @@
     </visual>
   </link>
+  <!-- ================ IMU ================= -->
   <joint name="imu_joint" type="fixed">
     <parent link="base_link"/>
@@ -56,4 +66,5 @@
   </joint>
   <link name="imu_link"/>
+  <!-- ================ LIDAR ================= -->
   <joint name="scan_joint" type="fixed">
     <parent link="base_link"/>
@@ -77,4 +88,5 @@
     </inertial>
   </link>
+  <!-- ================ CAMERA LINK ================= -->
   <joint name="camera_joint" type="fixed">
     <origin xyz="0.25 0.0 0.25" rpy="0 0.785398 0"/>
@@ -90,12 +102,6 @@
       <material name="dark"/>
     </visual>
-    <visual>
-      <origin xyz="0.015 0 0" rpy="0 1.57 0"/>
-      <geometry>
-        <cylinder length="0.03" radius="0.02"/>
-      </geometry>
-      <material name="dark"/>
-    </visual>
   </link>
+  <!-- ================ RGB CAMERA FRAMES ================= -->
   <joint name="camera_rgb_joint" type="fixed">
     <origin xyz="${r200_cam_rgb_px} ${r200_cam_rgb_py} ${r200_cam_rgb_pz}" rpy="0 0 0"/>
@@ -110,4 +116,5 @@
   </joint>
   <link name="camera_rgb_optical_frame"/>
+  <!-- ================ DEPTH CAMERA FRAMES ================= -->
   <joint name="camera_depth_joint" type="fixed">
     <origin xyz="${r200_cam_rgb_px} ${r200_cam_rgb_py + r200_cam_depth_offset} ${r200_cam_rgb_pz}" rpy="0 0 0"/>

Commit message: no gravity on parrot

File: src/description/urdf/parrot.urdf.xacro (robot description, xacro)
@@ -1,131 +1,175 @@
-<?xml version="1.0" ?>
+<?xml version="1.0"?>
 <robot name="parrot" xmlns:xacro="http://ros.org/wiki/xacro">
-  <!-- model name that Gazebo plugins will use for topics: /model/<model_name>/... -->
-  <xacro:arg name="model_name" default="drone1"/>
-  <!-- include local xacros from this package -->
-  <xacro:include filename="$(find description)/urdf/common_properties.urdf.xacro"/>
-  <xacro:include filename="$(find description)/urdf/parrot.gazebo.xacro"/>
-  <!-- camera offsets -->
-  <xacro:property name="r200_cam_rgb_px" value="0.005"/>
-  <xacro:property name="r200_cam_rgb_py" value="0.018"/>
-  <xacro:property name="r200_cam_rgb_pz" value="0.013"/>
-  <xacro:property name="r200_cam_depth_offset" value="0.01"/>
-  <!-- ================= base_link ================= -->
-  <link name="base_link">
-    <!-- inertia from original file -->
-    <inertial>
-      <origin xyz="0 0 0" rpy="0 0 0"/>
-      <mass value="0.503"/>
-      <inertia ixx="1.805e-3" ixy="-8.619e-7" ixz="1.555e-5"
-               iyy="1.764e-3" iyz="3.595e-7"
-               izz="3.328e-3" />
-    </inertial>
-    <!-- SIMPLE COLLISION so it doesn't fall through the world -->
-    <collision name="collision">
-      <origin xyz="0 0 0" rpy="0 0 0"/>
-      <geometry>
-        <box size="0.4 0.4 0.15"/>
-      </geometry>
-    </collision>
-    <!-- visuals (using your meshes copied into description/meshes) -->
-    <visual name="hull">
-      <geometry>
-        <mesh filename="file://$(find description)/meshes/hull.dae"/>
-      </geometry>
-    </visual>
-    <visual name="propeller_rr">
-      <origin xyz="-0.09035 -0.11423 -0.00501" rpy="0 0 0"/>
-      <geometry>
-        <mesh filename="file://$(find description)/meshes/propeller_rr.dae"/>
-      </geometry>
-    </visual>
-    <visual name="propeller_rl">
-      <origin xyz="0.09035 0.11452 -0.00501" rpy="0 0 0"/>
-      <geometry>
-        <mesh filename="file://$(find description)/meshes/propeller_rl.dae"/>
-      </geometry>
-    </visual>
-    <visual name="propeller_fr">
-      <origin xyz="0.08456 -0.11435 -0.00501" rpy="0 0 0"/>
-      <geometry>
-        <mesh filename="file://$(find description)/meshes/propeller_fr.dae"/>
-      </geometry>
-    </visual>
-    <visual name="propeller_fl">
-      <origin xyz="0.08456 0.11463 -0.00501" rpy="0 0 0"/>
-      <geometry>
-        <mesh filename="file://$(find description)/meshes/propeller_fl.dae"/>
-      </geometry>
-    </visual>
-  </link>
-  <!-- ================ IMU ================= -->
-  <joint name="imu_joint" type="fixed">
-    <parent link="base_link"/>
-    <child link="imu_link"/>
-    <origin xyz="0.0 0 0.068" rpy="0 0 0"/>
-  </joint>
-  <link name="imu_link"/>
-  <!-- ================ LIDAR ================= -->
-  <joint name="scan_joint" type="fixed">
-    <parent link="base_link"/>
-    <child link="base_scan"/>
-    <origin xyz="0 0 0.2" rpy="0 0 0"/>
-  </joint>
-  <link name="base_scan">
-    <visual>
-      <origin xyz="0 0 0" rpy="0 0 0"/>
-      <geometry>
-        <cylinder length="0.04" radius="0.09"/>
-      </geometry>
-      <material name="dark"/>
-    </visual>
-    <inertial>
-      <mass value="0" />
-      <origin xyz="0 0 0" />
-      <inertia ixx="0.001" ixy="0.0" ixz="0.0"
-               iyy="0.001" iyz="0.0"
-               izz="0.001" />
-    </inertial>
-  </link>
-  <!-- ================ CAMERA LINK ================= -->
-  <joint name="camera_joint" type="fixed">
-    <origin xyz="0.25 0.0 0.25" rpy="0 0.785398 0"/>
-    <parent link="base_link"/>
-    <child link="camera_link"/>
-  </joint>
-  <link name="camera_link">
-    <visual>
-      <origin xyz="0 0 0" rpy="0 0 0"/>
-      <geometry>
-        <box size="0.02 0.08 0.05"/>
-      </geometry>
-      <material name="dark"/>
-    </visual>
-  </link>
-  <!-- ================ RGB CAMERA FRAMES ================= -->
-  <joint name="camera_rgb_joint" type="fixed">
-    <origin xyz="${r200_cam_rgb_px} ${r200_cam_rgb_py} ${r200_cam_rgb_pz}" rpy="0 0 0"/>
-    <parent link="camera_link"/>
-    <child link="camera_rgb_frame"/>
-  </joint>
-  <link name="camera_rgb_frame"/>
-  <joint name="camera_rgb_optical_joint" type="fixed">
-    <origin xyz="0 0 0" rpy="-1.57 0 -1.57"/>
-    <parent link="camera_rgb_frame"/>
-    <child link="camera_rgb_optical_frame"/>
-  </joint>
-  <link name="camera_rgb_optical_frame"/>
-  <!-- ================ DEPTH CAMERA FRAMES ================= -->
-  <joint name="camera_depth_joint" type="fixed">
-    <origin xyz="${r200_cam_rgb_px} ${r200_cam_rgb_py + r200_cam_depth_offset} ${r200_cam_rgb_pz}" rpy="0 0 0"/>
-    <parent link="camera_link"/>
-    <child link="camera_depth_frame"/>
-  </joint>
-  <link name="camera_depth_frame"/>
-  <joint name="camera_depth_optical_joint" type="fixed">
-    <origin xyz="0 0 0" rpy="-1.57 0 -1.57"/>
-    <parent link="camera_depth_frame"/>
-    <child link="camera_depth_optical_frame"/>
-  </joint>
-  <link name="camera_depth_optical_frame"/>
+  <!-- visibility toggles from the original zip -->
+  <xacro:arg name="laser_visual"  default="false" />
+  <xacro:arg name="camera_visual" default="false"/>
+  <xacro:arg name="imu_visual"    default="false"/>
+  <!-- NEW: let us name the model so topics become /model/<name>/... -->
+  <xacro:arg name="model_name"    default="drone1"/>
+  <!-- keep the drone floating at its spawn height -->
+  <gazebo reference="base_link">
+    <gravity>0</gravity>
+  </gazebo>
+  <!-- IMU on imu_link -->
+  <gazebo reference="imu_link">
+    <sensor type="imu" name="imu">
+      <always_on>true</always_on>
+      <visualize>$(arg imu_visual)</visualize>
+      <update_rate>100</update_rate>
+      <topic>/model/$(arg model_name)/imu</topic>
+      <gz_frame_id>imu_link</gz_frame_id>
+      <imu>
+        <angular_velocity>
+          <x>
+            <noise type="gaussian">
+              <mean>0.0</mean>
+              <stddev>2e-4</stddev>
+              <bias_mean>0.0000075</bias_mean>
+              <bias_stddev>0.0000008</bias_stddev>
+            </noise>
+          </x>
+          <y>
+            <noise type="gaussian">
+              <mean>0.0</mean>
+              <stddev>2e-4</stddev>
+              <bias_mean>0.0000075</bias_mean>
+              <bias_stddev>0.0000008</bias_stddev>
+            </noise>
+          </y>
+          <z>
+            <noise type="gaussian">
+              <mean>0.0</mean>
+              <stddev>2e-4</stddev>
+              <bias_mean>0.0000075</bias_mean>
+              <bias_stddev>0.0000008</bias_stddev>
+            </noise>
+          </z>
+        </angular_velocity>
+        <linear_acceleration>
+          <x>
+            <noise type="gaussian">
+              <mean>0.0</mean>
+              <stddev>1.7e-2</stddev>
+              <bias_mean>0.1</bias_mean>
+              <bias_stddev>0.001</bias_stddev>
+            </noise>
+          </x>
+          <y>
+            <noise type="gaussian">
+              <mean>0.0</mean>
+              <stddev>1.7e-2</stddev>
+              <bias_mean>0.1</bias_mean>
+              <bias_stddev>0.001</bias_stddev>
+            </noise>
+          </y>
+          <z>
+            <noise type="gaussian">
+              <mean>0.0</mean>
+              <stddev>1.7e-2</stddev>
+              <bias_mean>0.1</bias_mean>
+              <bias_stddev>0.001</bias_stddev>
+            </noise>
+          </z>
+        </linear_acceleration>
+      </imu>
+      <plugin
+        filename="ignition-gazebo-imu-system"
+        name="ignition::gazebo::systems::Imu">
+      </plugin>
+    </sensor>
+    <material>Gazebo/Grey</material>
+  </gazebo>
+  <!-- Velocity control plugin (so we can drive it with /cmd_vel) -->
+  <gazebo>
+    <plugin
+      filename="ignition-gazebo-velocity-control-system"
+      name="ignition::gazebo::systems::VelocityControl">
+      <topic>/model/$(arg model_name)/cmd_vel</topic>
+    </plugin>
+  </gazebo>
+  <!-- Publish odometry separately -->
+  <gazebo>
+    <plugin
+      filename="ignition-gazebo-odometry-publisher-system"
+      name="ignition::gazebo::systems::OdometryPublisher">
+      <topic>/model/$(arg model_name)/odometry</topic>
+      <odom_publish_frequency>20</odom_publish_frequency>
+      <odom_frame>odom</odom_frame>
+      <robot_base_frame>base_link</robot_base_frame>
+    </plugin>
+  </gazebo>
+  <!-- Joint state publisher -->
+  <gazebo>
+    <plugin
+      filename="ignition-gazebo-joint-state-publisher-system"
+      name="ignition::gazebo::systems::JointStatePublisher">
+      <topic>/model/$(arg model_name)/joint_states</topic>
+    </plugin>
+  </gazebo>
+  <!-- Sensors plugin (for lidar/camera) -->
+  <gazebo>
+    <plugin
+        filename="libignition-gazebo-sensors-system.so"
+        name="ignition::gazebo::systems::Sensors">
+    </plugin>
+  </gazebo>
+  <!-- 2D lidar on base_scan -->
+  <gazebo reference="base_scan">
+    <material>Gazebo/FlatBlack</material>
+    <sensor type="gpu_lidar" name="lidar">
+      <pose relative_to="base_scan">0 0 0 0 0 0</pose>
+      <visualize>$(arg laser_visual)</visualize>
+      <topic>/model/$(arg model_name)/scan</topic>
+      <update_rate>3</update_rate>
+      <gz_frame_id>base_scan</gz_frame_id>
+      <ray>
+        <scan>
+          <horizontal>
+            <samples>360</samples>
+            <resolution>1</resolution>
+            <min_angle>0.0</min_angle>
+            <max_angle>6.28319</max_angle>
+          </horizontal>
+        </scan>
+        <range>
+          <min>0.2</min>
+          <max>40</max>
+          <resolution>0.015</resolution>
+        </range>
+        <noise>
+          <type>gaussian</type>
+          <mean>0.0</mean>
+          <stddev>0.01</stddev>
+        </noise>
+      </ray>
+      <always_on>true</always_on>
+    </sensor>
+  </gazebo>
+  <!-- RGBD camera on camera_link -->
+  <gazebo reference="camera_link">
+    <sensor name="rgbd_camera" type="rgbd_camera">
+      <camera>
+        <horizontal_fov>2.0944</horizontal_fov>
+        <image>
+          <width>720</width>
+          <height>480</height>
+        </image>
+        <clip>
+          <near>0.1</near>
+          <far>40</far>
+        </clip>
+        <depth_camera>
+          <clip>
+            <near>0.4</near>
+            <far>10</far>
+          </clip>
+        </depth_camera>
+      </camera>
+      <always_on>true</always_on>
+      <update_rate>3</update_rate>
+      <visualize>$(arg camera_visual)</visualize>
+      <topic>/model/$(arg model_name)/camera</topic>
+      <gz_frame_id>camera_link</gz_frame_id>
+    </sensor>
+  </gazebo>
 </robot>
